Commit message: add a floating camera to view the robot

File: ur_description/urdf/common.gazebo.xacro (robot description, xacro)
@@ -74,3 +74,56 @@
     </sensor>
   </gazebo>
+  <!-- external_camera_link -->
+  <gazebo reference="external_camera_link">
+    <mu1>0.2</mu1>
+    <mu2>0.2</mu2>
+    <material>Gazebo/Black</material>
+  </gazebo>
+ <!-- external camera -->
+  <gazebo reference="external_camera_link">
+    <sensor type="camera" name="camera1">
+      <update_rate>30.0</update_rate>
+      <camera name="head">
+        <horizontal_fov>1.3962634</horizontal_fov>
+        <image>
+          <width>800</width>
+          <height>800</height>
+          <format>R8G8B8</format>
+        </image>
+        <clip>
+          <near>0.02</near>
+          <far>300</far>
+        </clip>
+        <noise>
+          <type>gaussian</type>
+          <!-- Noise is sampled independently per pixel on each frame.
+               That pixel's noise value is added to each of its color
+               channels, which at that point lie in the range [0,1]. -->
+          <mean>0.0</mean>
+          <stddev>0.007</stddev>
+        </noise>
+      </camera>
+      <plugin name="camera_controller" filename="libgazebo_ros_camera.so">
+        <alwaysOn>true</alwaysOn>
+        <updateRate>0.0</updateRate>
+        <cameraName>external_cam</cameraName>
+        <imageTopicName>image_raw</imageTopicName>
+        <cameraInfoTopicName>camera_info</cameraInfoTopicName>
+        <frameName>camera_link_optical</frameName>
+        <!-- setting hackBaseline to anything but 0.0 will cause a misalignment
+            between the gazebo sensor image and the frame it is supposed to
+            be attached to -->
+        <hackBaseline>0.0</hackBaseline>
+        <distortionK1>0.0</distortionK1>
+        <distortionK2>0.0</distortionK2>
+        <distortionK3>0.0</distortionK3>
+        <distortionT1>0.0</distortionT1>
+        <distortionT2>0.0</distortionT2>
+        <CxPrime>0</CxPrime>
+        <Cx>0.0</Cx>
+        <Cy>0.0</Cy>
+        <focalLength>0.0</focalLength>
+      </plugin>
+    </sensor>
+  </gazebo>
 </robot>

File: ur_description/urdf/ur5.urdf.xacro (robot description, xacro)
@@ -381,4 +381,5 @@
       </plugin>
   </gazebo>
+  <!-- End Effector Camera -->
   <joint name="${prefix}camera_joint" type="fixed">
     <axis xyz="0 1 0" />
@@ -387,5 +388,4 @@
     <child link="${prefix}camera_link"/>
   </joint>
-  <!-- Camera -->
   <link name="${prefix}camera_link">
     <collision>
@@ -419,4 +419,42 @@
   <link name="${prefix}camera_link_optical">
   </link>
+  <!-- External Camera -->
+    <joint name="${prefix}external_camera_joint" type="fixed">
+    <axis xyz="0 1 0" />
+    <origin xyz="0.5 -0.8 0.9" rpy="${pi} ${pi*3/4} ${-pi/4}"/>
+    <parent link="${prefix}base_link"/>
+    <child link="${prefix}external_camera_link"/>
+  </joint>
+  <link name="${prefix}external_camera_link">
+    <collision>
+      <origin xyz="0 0 0" rpy="0 0 0"/>
+      <geometry>
+	<box size="${camera_link} ${camera_link} ${camera_link}"/>
+      </geometry>
+    </collision>
+    <visual>
+      <origin xyz="0 0 0" rpy="0 0 0"/>
+      <geometry>
+	<box size="${camera_link} ${camera_link} ${camera_link}"/>
+      </geometry>
+      <material name="green"/>
+    </visual>
+    <inertial>
+      <mass value="1e-5" />
+      <origin xyz="0 0 0" rpy="0 0 0"/>
+      <inertia ixx="1e-6" ixy="0" ixz="0" iyy="1e-6" iyz="0" izz="1e-6" />
+    </inertial>
+  </link>
+  <!-- generate an optical frame http://www.ros.org/reps/rep-0103.html#suffix-frames
+      so that ros and opencv can operate on the camera frame correctly -->
+  <joint name="${prefix}external_camera_optical_joint" type="fixed">
+    <!-- these values have to be these values otherwise the gazebo camera image
+        won't be aligned properly with the frame it is supposedly originating from -->
+    <origin xyz="0 0 0" rpy="${-pi/2} 0 ${-pi/2}"/>
+    <parent link="${prefix}external_camera_link"/>
+    <child link="${prefix}external_camera_link_optical"/>
+  </joint>
+  <link name="${prefix}external_camera_link_optical">
+  </link>
     <xacro:ur_arm_transmission prefix="${prefix}" hw_interface="hardware_interface/PositionJointInterface"/>
     <xacro:ur_arm_gazebo prefix="${prefix}" />

Commit message: add second camera

File: ur_description/urdf/common.gazebo.xacro (robot description, xacro)
@@ -34,6 +34,6 @@
         <horizontal_fov>1.3962634</horizontal_fov>
         <image>
-          <width>800</width>
-          <height>800</height>
+          <width>500</width>
+          <height>500</height>
           <format>R8G8B8</format>
         </image>
@@ -74,6 +74,6 @@
     </sensor>
   </gazebo>
-  <!-- external_camera_link -->
-  <gazebo reference="external_camera_link">
+  <!-- right_external_camera_link -->
+  <gazebo reference="right_external_camera_link">
     <mu1>0.2</mu1>
     <mu2>0.2</mu2>
@@ -81,5 +81,5 @@
   </gazebo>
  <!-- external camera -->
-  <gazebo reference="external_camera_link">
+  <gazebo reference="right_external_camera_link">
     <sensor type="camera" name="camera1">
       <update_rate>30.0</update_rate>
@@ -87,6 +87,6 @@
         <horizontal_fov>1.3962634</horizontal_fov>
         <image>
-          <width>800</width>
-          <height>800</height>
+          <width>500</width>
+          <height>500</height>
           <format>R8G8B8</format>
         </image>
@@ -107,5 +107,5 @@
         <alwaysOn>true</alwaysOn>
         <updateRate>0.0</updateRate>
-        <cameraName>external_cam</cameraName>
+        <cameraName>right_external_cam</cameraName>
         <imageTopicName>image_raw</imageTopicName>
         <cameraInfoTopicName>camera_info</cameraInfoTopicName>
@@ -127,3 +127,62 @@
     </sensor>
   </gazebo>
+    <!-- right_external_camera_link -->
+  <gazebo reference="right_external_camera_link">
+    <mu1>0.2</mu1>
+    <mu2>0.2</mu2>
+    <material>Gazebo/Black</material>
+  </gazebo>
+ <!-- left_external camera -->
+  <gazebo reference="left_external_camera_link">
+    <sensor type="camera" name="camera1">
+      <update_rate>30.0</update_rate>
+      <camera name="head">
+        <horizontal_fov>1.3962634</horizontal_fov>
+        <image>
+          <width>500</width>
+          <height>500</height>
+          <format>R8G8B8</format>
+        </image>
+        <clip>
+          <near>0.02</near>
+          <far>300</far>
+        </clip>
+        <noise>
+          <type>gaussian</type>
+          <!-- Noise is sampled independently per pixel on each frame.
+               That pixel's noise value is added to each of its color
+               channels, which at that point lie in the range [0,1]. -->
+          <mean>0.0</mean>
+          <stddev>0.007</stddev>
+        </noise>
+      </camera>
+      <plugin name="camera_controller" filename="libgazebo_ros_camera.so">
+        <alwaysOn>true</alwaysOn>
+        <updateRate>0.0</updateRate>
+        <cameraName>left_external_cam</cameraName>
+        <imageTopicName>image_raw</imageTopicName>
+        <cameraInfoTopicName>camera_info</cameraInfoTopicName>
+        <frameName>camera_link_optical</frameName>
+        <!-- setting hackBaseline to anything but 0.0 will cause a misalignment
+            between the gazebo sensor image and the frame it is supposed to
+            be attached to -->
+        <hackBaseline>0.0</hackBaseline>
+        <distortionK1>0.0</distortionK1>
+        <distortionK2>0.0</distortionK2>
+        <distortionK3>0.0</distortionK3>
+        <distortionT1>0.0</distortionT1>
+        <distortionT2>0.0</distortionT2>
+        <CxPrime>0</CxPrime>
+        <Cx>0.0</Cx>
+        <Cy>0.0</Cy>
+        <focalLength>0.0</focalLength>
+      </plugin>
+    </sensor>
+  </gazebo>
+  <!-- left_external_camera_link -->
+  <gazebo reference="left_external_camera_link">
+    <mu1>0.2</mu1>
+    <mu2>0.2</mu2>
+    <material>Gazebo/Black</material>
+  </gazebo>
 </robot>

File: ur_description/urdf/ur5.urdf.xacro (robot description, xacro)
@@ -419,12 +419,12 @@
   <link name="${prefix}camera_link_optical">
   </link>
-  <!-- External Camera -->
-    <joint name="${prefix}external_camera_joint" type="fixed">
+  <!-- Right External Camera -->
+    <joint name="${prefix}right_external_camera_joint" type="fixed">
     <axis xyz="0 1 0" />
     <origin xyz="0.5 -0.8 0.9" rpy="${pi} ${pi*3/4} ${-pi/4}"/>
     <parent link="${prefix}base_link"/>
-    <child link="${prefix}external_camera_link"/>
+    <child link="${prefix}right_external_camera_link"/>
   </joint>
-  <link name="${prefix}external_camera_link">
+  <link name="${prefix}right_external_camera_link">
     <collision>
       <origin xyz="0 0 0" rpy="0 0 0"/>
@@ -448,12 +448,50 @@
   <!-- generate an optical frame http://www.ros.org/reps/rep-0103.html#suffix-frames
       so that ros and opencv can operate on the camera frame correctly -->
-  <joint name="${prefix}external_camera_optical_joint" type="fixed">
+  <joint name="${prefix}right_external_camera_optical_joint" type="fixed">
     <!-- these values have to be these values otherwise the gazebo camera image
         won't be aligned properly with the frame it is supposedly originating from -->
     <origin xyz="0 0 0" rpy="${-pi/2} 0 ${-pi/2}"/>
-    <parent link="${prefix}external_camera_link"/>
-    <child link="${prefix}external_camera_link_optical"/>
+    <parent link="${prefix}right_external_camera_link"/>
+    <child link="${prefix}right_external_camera_link_optical"/>
   </joint>
-  <link name="${prefix}external_camera_link_optical">
+  <link name="${prefix}right_external_camera_link_optical">
+  </link>
+  <!-- Left External Camera -->
+    <joint name="${prefix}left_external_camera_joint" type="fixed">
+    <axis xyz="0 1 0" />
+    <origin xyz="-0.5 -0.8 0.9" rpy="${pi} ${pi*3/4} ${-pi*3/4}"/>
+    <parent link="${prefix}base_link"/>
+    <child link="${prefix}left_external_camera_link"/>
+  </joint>
+  <link name="${prefix}left_external_camera_link">
+    <collision>
+      <origin xyz="0 0 0" rpy="0 0 0"/>
+      <geometry>
+	<box size="${camera_link} ${camera_link} ${camera_link}"/>
+      </geometry>
+    </collision>
+    <visual>
+      <origin xyz="0 0 0" rpy="0 0 0"/>
+      <geometry>
+	<box size="${camera_link} ${camera_link} ${camera_link}"/>
+      </geometry>
+      <material name="green"/>
+    </visual>
+    <inertial>
+      <mass value="1e-5" />
+      <origin xyz="0 0 0" rpy="0 0 0"/>
+      <inertia ixx="1e-6" ixy="0" ixz="0" iyy="1e-6" iyz="0" izz="1e-6" />
+    </inertial>
+  </link>
+  <!-- generate an optical frame http://www.ros.org/reps/rep-0103.html#suffix-frames
+      so that ros and opencv can operate on the camera frame correctly -->
+  <joint name="${prefix}left_external_camera_optical_joint" type="fixed">
+    <!-- these values have to be these values otherwise the gazebo camera image
+        won't be aligned properly with the frame it is supposedly originating from -->
+    <origin xyz="0 0 0" rpy="${-pi/2} 0 ${-pi/2}"/>
+    <parent link="${prefix}left_external_camera_link"/>
+    <child link="${prefix}left_external_camera_link_optical"/>
+  </joint>
+  <link name="${prefix}left_external_camera_link_optical">
   </link>
     <xacro:ur_arm_transmission prefix="${prefix}" hw_interface="hardware_interface/PositionJointInterface"/>

Commit message: add laser pointer

File: ur_description/urdf/common.gazebo.xacro (robot description, xacro)
@@ -186,3 +186,25 @@
     <material>Gazebo/Black</material>
   </gazebo>
+  <gazebo reference="laser_link">
+    <projector name="projector_wg6802418">
+        <pose>0 0 0 0 0 0</pose>
+        <texture>dot.png</texture>
+        <fov>0.0125</fov>
+        <near_clip>.001</near_clip>
+        <far_clip>3</far_clip>
+     </projector>
+</gazebo>
+<gazebo>
+     <plugin name="projector" filename="libgazebo_ros_projector.so">
+         <projector>projector_wg6802418</projector>
+         <alwaysOn>true</alwaysOn>
+         <updateRate>10.0</updateRate>
+         <!-- Apparently the 2 lines below does not affect anything -->
+         <textureName></textureName>
+         <filterTextureName></filterTextureName>
+         <!-- end -->
+         <textureTopicName>/projector/image</textureTopicName>
+         <projectorTopicName>/projector/projector</projectorTopicName>
+     </plugin>
+</gazebo>
 </robot>

File: ur_description/urdf/ur5.urdf.xacro (robot description, xacro)
@@ -495,4 +495,23 @@
   <link name="${prefix}left_external_camera_link_optical">
   </link>
+  <joint name="${prefix}laser_joint" type="fixed">
+    <axis xyz="0 1 0" />
+    <origin rpy="${pi/-2} ${pi/-2} ${pi/2}" xyz="0.01 0.0125 0" />
+    <parent link="${prefix}ee_link"/>
+    <child link="${prefix}laser_link"/>
+  </joint>
+    <link name="laser_link">
+    <visual>
+      <origin xyz="0 0 0" rpy="0 0 0"/>
+      <geometry>
+        <box size="0.001 0.001 0.001"/>
+      </geometry>
+    </visual>
+    <inertial>
+      <mass value="1e-5" />
+      <origin xyz="0 0 0" rpy="0 0 0"/>
+      <inertia ixx="1e-6" ixy="0" ixz="0" iyy="1e-6" iyz="0" izz="1e-6" />
+    </inertial>
+  </link>
     <xacro:ur_arm_transmission prefix="${prefix}" hw_interface="hardware_interface/PositionJointInterface"/>
     <xacro:ur_arm_gazebo prefix="${prefix}" />
