Commit message: rotate camera so that away from base is up

File: ur_description/urdf/ur5.urdf.xacro (robot description, xacro)
@@ -656,5 +656,5 @@
   <joint name="camera_joint" type="fixed">
     <axis xyz="0 1 0" />
-    <origin xyz="-0.02 0.0 0.055" rpy="0 0 0"/>
+    <origin xyz="-0.02 0.0 0.055" rpy="${pi} 0 0"/>
     <parent link="ee_link"/>
     <child link="camera_link"/>

Commit message: use one rectangular (invisible) gripper

File: ur_description/urdf/ur5.urdf.xacro (robot description, xacro)
@@ -342,12 +342,22 @@
       <gravity>0</gravity>
       <visual>
-        <origin rpy="0 0 0" xyz="0 0 0"/>
-        <geometry>
-          <cylinder radius="0.005" length="0.01"/>
-        </geometry>
         <material name="transparent">
           <color rgba="0 0 0 0"/>
         </material>
       </visual>
+      <collision>
+        <origin rpy="0 0 -0.0375" xyz="0 0 0"/>
+        <geometry>
+          <box size="0.1 0.1 0.0375" />
+        </geometry>
+        <surface>
+          <friction>
+            <ode>
+              <mu>10</mu>
+              <mu2>10</mu2>
+            </ode>
+          </friction>
+        </surface>
+      </collision>
       <inertial>
         <origin rpy="0 0 0" xyz="0.000000 0.000000 0.000000"/>
@@ -369,289 +379,6 @@
         <bodyName>vacuum_gripper</bodyName>
         <topicName>grasping</topicName>
-	<maxForce>1</maxForce>
-        <maxDistance>0.05</maxDistance>
-        <minDistance>0.01</minDistance>
       </plugin>
   </gazebo>
-    <link name="vacuum_gripper1">
-      <gravity>0</gravity>
-      <visual>
-        <origin rpy="0 0 0" xyz="0 0 0"/>
-        <geometry>
-          <cylinder radius="0.005" length="0.01"/>
-        </geometry>
-        <material name="transparent">
-          <color rgba="0 0 0 0"/>
-        </material>
-      </visual>
-      <inertial>
-        <origin rpy="0 0 0" xyz="0.000000 0.000000 0.000000"/>
-        <mass value="0.0001"/>
-        <inertia ixx="1e-08" ixy="0" ixz="0" iyy="1e-08" iyz="0" izz="1e-08"/>
-      </inertial>
-    </link>
-    <joint name="gripper_joint1" type="revolute">
-      <axis xyz="1 0 0" />
-      <parent link="ee_link" />
-      <child link="vacuum_gripper1" />
-      <origin rpy="0 1.5708 0" xyz="0.01 -0.0125 0" />
-      <limit effort="50" velocity="50" lower="0" upper="0" />
-      <dynamics damping="0.0" friction="10"/>
-    </joint>
-  <gazebo>
-      <plugin name="gazebo_ros_vacuum_gripper1" filename="libgazebo_ros_vacuum_gripper.so">
-        <robotNamespace>/ur5/vacuum_gripper1</robotNamespace>
-        <bodyName>vacuum_gripper1</bodyName>
-        <topicName>grasping1</topicName>
-	<maxForce>1</maxForce>
-        <maxDistance>0.05</maxDistance>
-        <minDistance>0.01</minDistance>
-      </plugin>
-  </gazebo>
-    <link name="vacuum_gripper2">
-      <gravity>0</gravity>
-      <visual>
-        <origin rpy="0 0 0" xyz="0 0 0"/>
-        <geometry>
-          <cylinder radius="0.005" length="0.01"/>
-        </geometry>
-        <material name="transparent">
-          <color rgba="0 0 0 0"/>
-        </material>
-      </visual>
-      <inertial>
-        <origin rpy="0 0 0" xyz="0.000000 0.000000 0.000000"/>
-        <mass value="0.0001"/>
-        <inertia ixx="1e-08" ixy="0" ixz="0" iyy="1e-08" iyz="0" izz="1e-08"/>
-      </inertial>
-    </link>
-    <joint name="gripper_joint2" type="revolute">
-      <axis xyz="1 0 0" />
-      <parent link="ee_link" />
-      <child link="vacuum_gripper2" />
-      <origin rpy="0 1.5708 0" xyz="0.01 0 0.0125" />
-      <limit effort="50" velocity="50" lower="0" upper="0" />
-      <dynamics damping="0.0" friction="10"/>
-    </joint>
-  <gazebo>
-      <plugin name="gazebo_ros_vacuum_gripper2" filename="libgazebo_ros_vacuum_gripper.so">
-        <robotNamespace>/ur5/vacuum_gripper2</robotNamespace>
-        <bodyName>vacuum_gripper2</bodyName>
-        <topicName>grasping2</topicName>
-	<maxForce>1</maxForce>
-        <maxDistance>0.05</maxDistance>
-        <minDistance>0.01</minDistance>
-      </plugin>
-  </gazebo>
-    <link name="vacuum_gripper3">
-      <gravity>0</gravity>
-      <visual>
-        <origin rpy="0 0 0" xyz="0 0 0"/>
-        <geometry>
-          <cylinder radius="0.005" length="0.01"/>
-        </geometry>
-        <material name="transparent">
-          <color rgba="0 0 0 0"/>
-        </material>
-      </visual>
-      <inertial>
-        <origin rpy="0 0 0" xyz="0.000000 0.000000 0.000000"/>
-        <mass value="0.0001"/>
-        <inertia ixx="1e-08" ixy="0" ixz="0" iyy="1e-08" iyz="0" izz="1e-08"/>
-      </inertial>
-    </link>
-    <joint name="gripper_joint3" type="revolute">
-      <axis xyz="1 0 0" />
-      <parent link="ee_link" />
-      <child link="vacuum_gripper3" />
-      <origin rpy="0 1.5708 0" xyz="0.01 0 -0.0125" />
-      <limit effort="50" velocity="50" lower="0" upper="0" />
-      <dynamics damping="0.0" friction="10"/>
-    </joint>
-  <gazebo>
-      <plugin name="gazebo_ros_vacuum_gripper3" filename="libgazebo_ros_vacuum_gripper.so">
-        <robotNamespace>/ur5/vacuum_gripper3</robotNamespace>
-        <bodyName>vacuum_gripper3</bodyName>
-        <topicName>grasping2</topicName>
-	<maxForce>1</maxForce>
-        <maxDistance>0.05</maxDistance>
-        <minDistance>0.01</minDistance>
-      </plugin>
-  </gazebo>
-  <link name="vacuum_gripper4">
-    <gravity>0</gravity>
-    <visual>
-      <origin rpy="0 0 0" xyz="0 0 0"/>
-      <geometry>
-        <cylinder radius="0.005" length="0.01"/>
-      </geometry>
-      <material name="transparent">
-        <color rgba="0 0 0 0"/>
-      </material>
-    </visual>
-    <inertial>
-      <origin rpy="0 0 0" xyz="0.000000 0.000000 0.000000"/>
-      <mass value="0.0001"/>
-      <inertia ixx="1e-08" ixy="0" ixz="0" iyy="1e-08" iyz="0" izz="1e-08"/>
-    </inertial>
-  </link>
-  <joint name="gripper_joint4" type="revolute">
-    <axis xyz="1 0 0" />
-    <parent link="ee_link" />
-    <child link="vacuum_gripper4" />
-    <origin rpy="0 1.5708 0" xyz="0.01 0 0" />
-    <limit effort="50" velocity="50" lower="0" upper="0" />
-    <dynamics damping="0.0" friction="10"/>
-  </joint>
-  <gazebo>
-    <plugin name="gazebo_ros_vacuum_gripper4" filename="libgazebo_ros_vacuum_gripper.so">
-      <robotNamespace>/ur5/vacuum_gripper4</robotNamespace>
-      <bodyName>vacuum_gripper4</bodyName>
-      <topicName>grasping4</topicName>
-  <maxForce>1</maxForce>
-      <maxDistance>0.05</maxDistance>
-      <minDistance>0.01</minDistance>
-    </plugin>
-  </gazebo>
-  <link name="vacuum_gripper5">
-    <gravity>0</gravity>
-    <visual>
-      <origin rpy="0 0 0" xyz="0 0 0"/>
-      <geometry>
-        <cylinder radius="0.005" length="0.01"/>
-      </geometry>
-      <material name="transparent">
-        <color rgba="0 0 0 0"/>
-      </material>
-    </visual>
-    <inertial>
-      <origin rpy="0 0 0" xyz="0.000000 0.000000 0.000000"/>
-      <mass value="0.0001"/>
-      <inertia ixx="1e-08" ixy="0" ixz="0" iyy="1e-08" iyz="0" izz="1e-08"/>
-    </inertial>
-  </link>
-  <joint name="gripper_joint5" type="revolute">
-    <axis xyz="1 0 0" />
-    <parent link="ee_link" />
-    <child link="vacuum_gripper5" />
-    <origin rpy="0 1.5708 0" xyz="0.01 0.0125 0.0125" />
-    <limit effort="50" velocity="50" lower="0" upper="0" />
-    <dynamics damping="0.0" friction="10"/>
-  </joint>
-<gazebo>
-    <plugin name="gazebo_ros_vacuum_gripper" filename="libgazebo_ros_vacuum_gripper.so">
-      <robotNamespace>/ur5/vacuum_gripper5</robotNamespace>
-      <bodyName>vacuum_gripper5</bodyName>
-      <topicName>grasping5</topicName>
-<maxForce>1</maxForce>
-      <maxDistance>0.05</maxDistance>
-      <minDistance>0.01</minDistance>
-    </plugin>
-</gazebo>
-  <link name="vacuum_gripper6">
-    <gravity>0</gravity>
-    <visual>
-      <origin rpy="0 0 0" xyz="0 0 0"/>
-      <geometry>
-        <cylinder radius="0.005" length="0.01"/>
-      </geometry>
-      <material name="transparent">
-        <color rgba="0 0 0 0"/>
-      </material>
-    </visual>
-    <inertial>
-      <origin rpy="0 0 0" xyz="0.000000 0.000000 0.000000"/>
-      <mass value="0.0001"/>
-      <inertia ixx="1e-08" ixy="0" ixz="0" iyy="1e-08" iyz="0" izz="1e-08"/>
-    </inertial>
-  </link>
-  <joint name="gripper_joint6" type="revolute">
-    <axis xyz="1 0 0" />
-    <parent link="ee_link" />
-    <child link="vacuum_gripper6" />
-    <origin rpy="0 1.5708 0" xyz="0.01 -0.0125 0.0125" />
-    <limit effort="50" velocity="50" lower="0" upper="0" />
-    <dynamics damping="0.0" friction="10"/>
-  </joint>
-<gazebo>
-    <plugin name="gazebo_ros_vacuum_gripper1" filename="libgazebo_ros_vacuum_gripper.so">
-      <robotNamespace>/ur5/vacuum_gripper6</robotNamespace>
-      <bodyName>vacuum_gripper6</bodyName>
-      <topicName>grasping6</topicName>
-<maxForce>1</maxForce>
-      <maxDistance>0.05</maxDistance>
-      <minDistance>0.01</minDistance>
-    </plugin>
-</gazebo>
-  <link name="vacuum_gripper7">
-    <gravity>0</gravity>
-    <visual>
-      <origin rpy="0 0 0" xyz="0 0 0"/>
-      <geometry>
-        <cylinder radius="0.005" length="0.01"/>
-      </geometry>
-      <material name="transparent">
-        <color rgba="0 0 0 0"/>
-      </material>
-    </visual>
-    <inertial>
-      <origin rpy="0 0 0" xyz="0.000000 0.000000 0.000000"/>
-      <mass value="0.0001"/>
-      <inertia ixx="1e-08" ixy="0" ixz="0" iyy="1e-08" iyz="0" izz="1e-08"/>
-    </inertial>
-  </link>
-  <joint name="gripper_joint7" type="revolute">
-    <axis xyz="1 0 0" />
-    <parent link="ee_link" />
-    <child link="vacuum_gripper7" />
-    <origin rpy="0 1.5708 0" xyz="0.01 0.0125 -0.0125" />
-    <limit effort="50" velocity="50" lower="0" upper="0" />
-    <dynamics damping="0.0" friction="10"/>
-  </joint>
-<gazebo>
-    <plugin name="gazebo_ros_vacuum_gripper7" filename="libgazebo_ros_vacuum_gripper.so">
-      <robotNamespace>/ur5/vacuum_gripper7</robotNamespace>
-      <bodyName>vacuum_gripper7</bodyName>
-      <topicName>grasping7</topicName>
-<maxForce>1</maxForce>
-      <maxDistance>0.05</maxDistance>
-      <minDistance>0.01</minDistance>
-    </plugin>
-</gazebo>
-  <link name="vacuum_gripper8">
-    <gravity>0</gravity>
-    <visual>
-      <origin rpy="0 0 0" xyz="0 0 0"/>
-      <geometry>
-        <cylinder radius="0.005" length="0.01"/>
-      </geometry>
-      <material name="transparent">
-        <color rgba="0 0 0 0"/>
-      </material>
-    </visual>
-    <inertial>
-      <origin rpy="0 0 0" xyz="0.000000 0.000000 0.000000"/>
-      <mass value="0.0001"/>
-      <inertia ixx="1e-08" ixy="0" ixz="0" iyy="1e-08" iyz="0" izz="1e-08"/>
-    </inertial>
-  </link>
-  <joint name="gripper_joint8" type="revolute">
-    <axis xyz="1 0 0" />
-    <parent link="ee_link" />
-    <child link="vacuum_gripper8" />
-    <origin rpy="0 1.5708 0" xyz="0.01 -0.0125 -0.0125" />
-    <limit effort="50" velocity="50" lower="0" upper="0" />
-    <dynamics damping="0.0" friction="10"/>
-  </joint>
-<gazebo>
-    <plugin name="gazebo_ros_vacuum_gripper8" filename="libgazebo_ros_vacuum_gripper.so">
-      <robotNamespace>/ur5/vacuum_gripper8</robotNamespace>
-      <bodyName>vacuum_gripper8</bodyName>
-      <topicName>grasping8</topicName>
-<maxForce>1</maxForce>
-      <maxDistance>0.05</maxDistance>
-      <minDistance>0.01</minDistance>
-    </plugin>
-</gazebo>
   <joint name="camera_joint" type="fixed">
     <axis xyz="0 1 0" />

Commit message: add gripper_prefix and plumb through it and existing prefix

File: ur_description/urdf/ur5.urdf.xacro (robot description, xacro)
@@ -12,5 +12,5 @@
     </inertial>
   </xacro:macro>
-  <xacro:macro name="ur5_robot" params="prefix joint_limited
+  <xacro:macro name="ur5_robot" params="prefix gripper_prefix joint_limited
     shoulder_pan_lower_limit:=${-pi}    shoulder_pan_upper_limit:=${pi}
     shoulder_lift_lower_limit:=${-pi}    shoulder_lift_upper_limit:=${pi}
@@ -339,5 +339,5 @@
       </collision>
     </link>
-    <link name="vacuum_gripper">
+    <link name="${prefix}vacuum_gripper">
       <gravity>0</gravity>
       <visual>
@@ -366,8 +366,8 @@
       </inertial>
     </link>
-    <joint name="gripper_joint" type="revolute">
+    <joint name="${prefix}gripper_joint" type="revolute">
       <axis xyz="1 0 0" />
-      <parent link="ee_link" />
-      <child link="vacuum_gripper" />
+      <parent link="${prefix}ee_link" />
+      <child link="${prefix}vacuum_gripper" />
       <origin rpy="0 1.5708 0" xyz="0.01 0.0125 0" />
       <limit effort="50" velocity="50" lower="0" upper="0" />
@@ -375,18 +375,18 @@
     </joint>
   <gazebo>
-      <plugin name="gazebo_ros_vacuum_gripper" filename="libgripper.so">
-        <robotNamespace>/ur5/vacuum_gripper</robotNamespace>
-        <bodyName>vacuum_gripper</bodyName>
-        <topicName>grasping</topicName>
+      <plugin name="${prefix}gazebo_ros_vacuum_gripper" filename="libgripper.so">
+        <robotNamespace>/${gripper_prefix}ur5/vacuum_gripper</robotNamespace>
+        <bodyName>${prefix}vacuum_gripper</bodyName>
+        <topicName>${prefix}grasping</topicName>
       </plugin>
   </gazebo>
-  <joint name="camera_joint" type="fixed">
+  <joint name="${prefix}camera_joint" type="fixed">
     <axis xyz="0 1 0" />
     <origin xyz="-0.02 0.0 0.055" rpy="${pi} 0 0"/>
-    <parent link="ee_link"/>
-    <child link="camera_link"/>
+    <parent link="${prefix}ee_link"/>
+    <child link="${prefix}camera_link"/>
   </joint>
   <!-- Camera -->
-  <link name="camera_link">
+  <link name="${prefix}camera_link">
     <collision>
       <origin xyz="0 0 0" rpy="0 0 0"/>
@@ -410,12 +410,12 @@
   <!-- generate an optical frame http://www.ros.org/reps/rep-0103.html#suffix-frames
       so that ros and opencv can operate on the camera frame correctly -->
-  <joint name="camera_optical_joint" type="fixed">
+  <joint name="${prefix}camera_optical_joint" type="fixed">
     <!-- these values have to be these values otherwise the gazebo camera image
         won't be aligned properly with the frame it is supposedly originating from -->
     <origin xyz="0 0 0" rpy="${-pi/2} 0 ${-pi/2}"/>
-    <parent link="camera_link"/>
-    <child link="camera_link_optical"/>
+    <parent link="${prefix}camera_link"/>
+    <child link="${prefix}camera_link_optical"/>
   </joint>
-  <link name="camera_link_optical">
+  <link name="${prefix}camera_link_optical">
   </link>
     <xacro:ur_arm_transmission prefix="${prefix}" hw_interface="hardware_interface/PositionJointInterface"/>

File: ur_description/urdf/ur5_robot.urdf.xacro (robot description, xacro)
@@ -3,4 +3,6 @@
        name="ur5" >
   <xacro:arg name="transmission_hw_interface" default="hardware_interface/PositionJointInterface"/>
+  <xacro:arg name="prefix" default=""/>
+  <xacro:arg name="gripper_prefix" default=""/>
   <!-- common stuff -->
   <xacro:include filename="$(find ur_description)/urdf/common.gazebo.xacro" />
@@ -8,5 +10,5 @@
   <xacro:include filename="$(find ur_description)/urdf/ur5.urdf.xacro" />
   <!-- arm -->
-  <xacro:ur5_robot prefix="" joint_limited="false"
+  <xacro:ur5_robot prefix="$(arg prefix)" gripper_prefix="$(arg gripper_prefix)" joint_limited="false"
     transmission_hw_interface="$(arg transmission_hw_interface)"
   />
@@ -14,5 +16,5 @@
   <joint name="world_joint" type="fixed">
     <parent link="world" />
-    <child link = "base_link" />
+    <child link = "$(arg prefix)base_link" />
     <origin xyz="0.0 0.0 0.0" rpy="0.0 0.0 0.0" />
   </joint>

Commit message: shift external camera locations

File: ur_description/urdf/ur5.urdf.xacro (robot description, xacro)
@@ -422,5 +422,5 @@
     <joint name="${prefix}right_external_camera_joint" type="fixed">
     <axis xyz="0 1 0" />
-    <origin xyz="0.5 -0.8 0.9" rpy="${pi} ${pi*3/4} ${-pi/4}"/>
+    <origin xyz="0.7 -0.7 0.9" rpy="${pi} ${pi*3/4} ${-pi/4}"/>
     <parent link="${prefix}base_link"/>
     <child link="${prefix}right_external_camera_link"/>
@@ -460,5 +460,5 @@
     <joint name="${prefix}left_external_camera_joint" type="fixed">
     <axis xyz="0 1 0" />
-    <origin xyz="-0.5 -0.8 0.9" rpy="${pi} ${pi*3/4} ${-pi*3/4}"/>
+    <origin xyz="-0.7 -0.7 0.9" rpy="${pi} ${pi*3/4} ${-pi*3/4}"/>
     <parent link="${prefix}base_link"/>
     <child link="${prefix}left_external_camera_link"/>

Commit message: removed visual for gripper. griper joint is fixed.

File: ur_description/urdf/ur5.urdf.xacro (robot description, xacro)
@@ -341,9 +341,4 @@
     <link name="${prefix}vacuum_gripper">
       <gravity>0</gravity>
-      <visual>
-        <material name="transparent">
-          <color rgba="0 0 0 0"/>
-        </material>
-      </visual>
       <collision>
         <origin rpy="0 0 -0.0375" xyz="0 0 0"/>
@@ -366,11 +361,11 @@
       </inertial>
     </link>
-    <joint name="${prefix}gripper_joint" type="revolute">
+    <joint name="${prefix}gripper_joint" type="fixed">
       <axis xyz="1 0 0" />
       <parent link="${prefix}ee_link" />
       <child link="${prefix}vacuum_gripper" />
       <origin rpy="0 1.5708 0" xyz="0.01 0.0125 0" />
-      <limit effort="50" velocity="50" lower="0" upper="0" />
-      <dynamics damping="0.0" friction="10"/>
+      <!-- <limit effort="50" velocity="50" lower="0" upper="0" />
+      <dynamics damping="0.0" friction="10"/> -->
     </joint>
   <gazebo>
